File: esquematico_Zynq-UltraScale/esquematico_Zynq-UltraScale/PINOUT.sch (KiCad schematic (older format))
At the start: 41 parts, among them Q1 PN2222A, Q2 PN2222A, Q3 PN2222A, Q4 PN2222A, Q5 PN2222A, Q6 PN2222A, Q7 PN2222A, Q8 PN2222A, SW2 SW_Push, SW3 SW_Push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

Commit message: upd
Parts:
- removed Q1, Q2, Q3, Q4, Q5, Q6, Q7, Q8: PN2222A, Package_TO_SOT_THT:TO-92_Inline, symbol Transistor_BJT:PN2222A
- added Q? (x8): NDS331N, symbol Zynq_UltraScale:NDS331N
Connections:
- net +3V3: now also D2.2 (A), D3.2 (A), D4.2 (A), D5.2 (A), D6.2 (A), D7.2 (A), D8.2 (A), D9.2 (A)
- net GND: now also Q?.2 (S), Q?.2 (S), Q?.2 (S), Q?.2 (S), Q?.2 (S), Q?.2 (S), Q?.2 (S), Q?.2 (S); no longer D2.1 (K), D3.1 (K), D4.1 (K), D5.1 (K), D6.1 (K), D7.1 (K), D8.1 (K), D9.1 (K)
- net LED_0: now also Q?.1 (G)
- net LED_1: now also Q?.1 (G)
- net LED_2: now also Q?.1 (G)
- net LED_3: now also Q?.1 (G)
- net LED_4: now also Q?.1 (G)
- net LED_5: now also Q?.1 (G)
- net LED_6: now also Q?.1 (G)
- net LED_7: now also Q?.1 (G)
- net at R94.2: now also D2.1 (K); no longer D2.2 (A)
- net at R94.1: now also Q?.3 (D)
- net at R95.2: now also D3.1 (K); no longer D3.2 (A)
- net at R95.1: now also Q?.3 (D)
- net at R96.2: now also D4.1 (K); no longer D4.2 (A)
- net at R96.1: now also Q?.3 (D)
- net at R99.2: now also D5.1 (K); no longer D5.2 (A)
- net at R99.1: now also Q?.3 (D)
- net at R101.2: now also D6.1 (K); no longer D6.2 (A)
- net at R101.1: now also Q?.3 (D)
- net at R103.2: now also D7.1 (K); no longer D7.2 (A)
- net at R103.1: now also Q?.3 (D)
- net at R106.2: now also D8.1 (K); no longer D8.2 (A)
- net at R106.1: now also Q?.3 (D)
- net at R109.2: now also D9.1 (K); no longer D9.2 (A)
- net at R109.1: now also Q?.3 (D)
Other:
- moved on the sheet: D2, D3, D4, D5, D6, D7, D8, D9, R101, R103, R106, R109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

Commit message: update
Parts:
- gave numbers to parts that had none: 8
Changed lines of the file:
@@
 LED_1
 $Comp
-L Zynq_UltraScale:NDS331N Q?
+L Zynq_UltraScale:NDS331N Q1
 U 1 1 613AF7D2
 P 5050 2150
-F 0 "Q?" H 5255 2196 50  0000 L CNN
+F 0 "Q1" H 5255 2196 50  0000 L CNN
 F 1 "NDS331N" H 5255 2105 50  0000 L CNN
 F 2 "" H 5250 2075 50  0001 L CIN
@@
 $EndComp
 $Comp
-L Zynq_UltraScale:NDS331N Q?
+L Zynq_UltraScale:NDS331N Q2
 U 1 1 613B14C9
 P 5850 2150
-F 0 "Q?" H 6055 2196 50  0000 L CNN
+F 0 "Q2" H 6055 2196 50  0000 L CNN
 F 1 "NDS331N" H 6055 2105 50  0000 L CNN
 F 2 "" H 6050 2075 50  0001 L CIN
@@
 $EndComp
 $Comp
-L Zynq_UltraScale:NDS331N Q?
+L Zynq_UltraScale:NDS331N Q3
 U 1 1 613B2347
 P 6650 2150
-F 0 "Q?" H 6855 2196 50  0000 L CNN
+F 0 "Q3" H 6855 2196 50  0000 L CNN
 F 1 "NDS331N" H 6855 2105 50  0000 L CNN
 F 2 "" H 6850 2075 50  0001 L CIN
@@
 $EndComp
 $Comp
-L Zynq_UltraScale:NDS331N Q?
+L Zynq_UltraScale:NDS331N Q4
 U 1 1 613B33DB
 P 7450 2150
-F 0 "Q?" H 7655 2196 50  0000 L CNN
+F 0 "Q4" H 7655 2196 50  0000 L CNN
 F 1 "NDS331N" H 7655 2105 50  0000 L CNN
 F 2 "" H 7650 2075 50  0001 L CIN
@@
 $EndComp
 $Comp
-L Zynq_UltraScale:NDS331N Q?
+L Zynq_UltraScale:NDS331N Q5
 U 1 1 613B3F87
 P 8250 2150
-F 0 "Q?" H 8455 2196 50  0000 L CNN
+F 0 "Q5" H 8455 2196 50  0000 L CNN
 F 1 "NDS331N" H 8455 2105 50  0000 L CNN
 F 2 "" H 8450 2075 50  0001 L CIN
@@
 $EndComp
 $Comp
-L Zynq_UltraScale:NDS331N Q?
+L Zynq_UltraScale:NDS331N Q6
 U 1 1 613B5A6B
 P 9050 2150
-F 0 "Q?" H 9255 2196 50  0000 L CNN
+F 0 "Q6" H 9255 2196 50  0000 L CNN
 F 1 "NDS331N" H 9255 2105 50  0000 L CNN
 F 2 "" H 9250 2075 50  0001 L CIN
@@
 $EndComp
 $Comp
-L Zynq_UltraScale:NDS331N Q?
+L Zynq_UltraScale:NDS331N Q7
 U 1 1 613B708A
 P 9850 2150
-F 0 "Q?" H 10055 2196 50  0000 L CNN
+F 0 "Q7" H 10055 2196 50  0000 L CNN
 F 1 "NDS331N" H 10055 2105 50  0000 L CNN
 F 2 "" H 10050 2075 50  0001 L CIN
@@
 $EndComp
 $Comp
-L Zynq_UltraScale:NDS331N Q?
+L Zynq_UltraScale:NDS331N Q8
 U 1 1 613B83B9
 P 10650 2150
-F 0 "Q?" H 10855 2196 50  0000 L CNN
+F 0 "Q8" H 10855 2196 50  0000 L CNN
 F 1 "NDS331N" H 10855 2105 50  0000 L CNN
 F 2 "" H 10850 2075 50  0001 L CIN
