File: esquematico_Zynq-UltraScale/esquematico_Zynq-UltraScale/alimentaciones.sch (KiCad schematic (older format))
At the start: 49 parts, among them J1 , SW1 SW_SPST, U1 TPS563201, U2 TPS563201, U3 TPS563201, U4 TPS563201, U5 XCZU2CG

Commit message: upd
Connections:
- net +1V8: now also U5.AA5 (VCCO_PSIO0_500), U5.C11 (VCCO_PSIO1_501), U5.C16 (VCCO_PSIO2_502), U5.D14 (VCCO_PSIO2_502), U5.F10 (VCCO_PSIO1_501), U5.G13 (VCCO_PSIO3_503), U5.H16 (VCCO_PSIO3_503), U5.V6 (VCCO_PSIO0_500)
- net +3V3: no longer U5.AA5 (VCCO_PSIO0_500), U5.C11 (VCCO_PSIO1_501), U5.C16 (VCCO_PSIO2_502), U5.D14 (VCCO_PSIO2_502), U5.F10 (VCCO_PSIO1_501), U5.G13 (VCCO_PSIO3_503), U5.H16 (VCCO_PSIO3_503), U5.V6 (VCCO_PSIO0_500)
Changed lines of the file:
@@
 Wire Wire Line
 	14100 3050 14550 3050
-$Comp
-L power:+3V3 #PWR0107
-U 1 1 61339441
-P 14600 3550
-F 0 "#PWR0107" H 14600 3400 50  0001 C CNN
-F 1 "+3V3" V 14600 3678 50  0000 L CNN
-F 2 "" H 14600 3550 50  0001 C CNN
-F 3 "" H 14600 3550 50  0001 C CNN
-	1    14600 3550
-	0    1    1    0
-$EndComp
 Wire Wire Line
 	14300 3550 14600 3550
@@
 	0    1    1    0
 $EndComp
+$Comp
+L power:+1V8 #PWR?
+U 1 1 61657550
+P 14600 3550
+F 0 "#PWR?" H 14600 3400 50  0001 C CNN
+F 1 "+1V8" V 14615 3678 50  0000 L CNN
+F 2 "" H 14600 3550 50  0001 C CNN
+F 3 "" H 14600 3550 50  0001 C CNN
+	1    14600 3550
+	0    1    1    0
+$EndComp
