File: esquematico_Zynq-UltraScale/esquematico_Zynq-UltraScale/esquematico_Zynq-UltraScale.kicad_pcb (KiCad board)
At the start: 2 copper layers, 13 parts, among them Q1 PN2222A, Q2 PN2222A, Q3 PN2222A, Q4 PN2222A, Q5 PN2222A, Q6 PN2222A, Q7 PN2222A, Q8 PN2222A, U5 XCZU2CG, U6 MT40A512M16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

Commit message: update
Parts:
- removed Q1, Q2, Q3, Q4, Q5, Q6, Q7, Q8: PN2222A, Package_TO_SOT_THT:TO-92_Inline
- added U10: MT25QU512ABB, Zynq-eame_UltraScale_0:BGA-25_5x5_6.0x8.0mm, F.Cu at (78.8, 61.2)
- U9: value FT2232HL -> IP4856CX25; footprint Package_QFP:LQFP-64_10x10mm_P0.5mm -> Zynq-eame_UltraScale_0:BGA-25_5x5_2.049999x2.049999mm
- moved U9 33.6 mm to (84.3, 58.2)
Connections:
- U5 pad A11: (no net) -> /MIO & REFERENCIA/MIO_CD
- U5 pad A12: (no net) -> /MIO & REFERENCIA/MIO_DAT2
- U5 pad A13: (no net) -> /MIO & REFERENCIA/MIO_CMD
- U5 pad A6: /PINOUT/LED_0 -> (no net)
- U5 pad A7: /PINOUT/LED_4 -> (no net)
- U5 pad A8: /PINOUT/LED_5 -> (no net)
- U5 pad A9: /PINOUT/LED_6 -> (no net)
- U5 pad AA1: (no net) -> /MIO & REFERENCIA/CS
- U5 pad AA5: +3V3 -> +1V8
- U5 pad B10: (no net) -> /MIO & REFERENCIA/MIO_DIR0
- U5 pad B11: (no net) -> /MIO & REFERENCIA/MIO_WP
- U5 pad B12: (no net) -> /MIO & REFERENCIA/MIO_DAT1
- U5 pad B5: /PINOUT/LED_2 -> (no net)
- U5 pad B6: /PINOUT/LED_3 -> (no net)
- U5 pad B7: /PINOUT/LED_1 -> (no net)
- U5 pad B9: /PINOUT/LED_7 -> (no net)
- U5 pad C10: (no net) -> /MIO & REFERENCIA/MIO_SEL
- U5 pad C11: +3V3 -> +1V8
- U5 pad C12: (no net) -> /MIO & REFERENCIA/MIO_DAT0
- U5 pad C13: (no net) -> /MIO & REFERENCIA/MIO_CLK_IN
- U5 pad C16: +3V3 -> +1V8
- U5 pad D11: (no net) -> /MIO & REFERENCIA/MIO_DIR_CMD
- U5 pad D12: (no net) -> /MIO & REFERENCIA/MIO_DIR1_3
- U5 pad D13: (no net) -> /MIO & REFERENCIA/MIO_DAT3
- U5 pad D14: +3V3 -> +1V8
- U5 pad F10: +3V3 -> +1V8
- U5 pad G13: +3V3 -> +1V8
- U5 pad H15: (no net) -> GND
- U5 pad H16: +3V3 -> +1V8
- U5 pad H18: (no net) -> GND
- U5 pad J15: (no net) -> GND
- U5 pad J16: (no net) -> GND
- U5 pad U4: (no net) -> /MIO & REFERENCIA/SCK
- U5 pad U5: (no net) -> /MIO & REFERENCIA/IO3
- U5 pad U6: (no net) -> /MIO & REFERENCIA/IO0
- U5 pad V2: (no net) -> /MIO & REFERENCIA/IO2
- U5 pad V3: /MIO & REFERENCIA/TX -> (no net)
- U5 pad V5: /MIO & REFERENCIA/RX -> (no net)
- U5 pad V6: +3V3 -> +1V8
- U5 pad W1: (no net) -> /MIO & REFERENCIA/IO1
