File: esquematico_Zynq-UltraScale/esquematico_Zynq-UltraScale/MIO_REFERENCIA.sch (KiCad schematic (older format))
At the start: 52 parts, among them J2 , J3 , J4 Conn_01x05, SW10 SW_Push, U10 TPS3106K33DBV, U11 S25FL128S, U5 XCZU2CG, U8 93C46, U9 FT2232HL, X1 ASE-xxxMHz, Y1 12MHz

Commit message: upd
Parts:
- removed C48, C50: 4.7uF, symbol Device:CP1
- removed C49, C51, C54, C56, C57, C59, C60, C63: 100nF, symbol Device:C
- removed C52, C58: 27pF, symbol Device:C
- removed C55: 3.3uF, symbol Device:C
- removed L5, L6: (no value), symbol Device:L_Core_Iron
- removed R111: 360, symbol Device:R_US
- removed R114: 2k2, symbol Device:R_US
- removed R128, R129, R130: 10k, symbol Device:R_US
- removed U11: S25FL128S, ZYNQ_7000:S03016-(SOIC-16), symbol Zynq_7000:S25FL128S
- removed U8: 93C46, symbol Zynq_7000:93C46
- removed U9: FT2232HL, Package_QFP:LQFP-64_10x10mm_P0.5mm, symbol Interface_USB:FT2232HL
- removed Y1: 12MHz, symbol Device:Crystal
- added C?: 100nF, symbol Device:C
- added C? (x2): 18pF, symbol Device:C
- added R?: 200, symbol Device:R_US
- added R?: 10K, symbol Device:R_US
- added U?: MT25QU512ABB, Zynq-eame_UltraScale_0:BGA-25_5x5_6.0x8.0mm, symbol Zynq_UltraScale:MT25QU512ABB
- added U?: IP4856CX25, Zynq-eame_UltraScale_0:BGA-25_5x5_2.049999x2.049999mm, symbol Zynq_UltraScale:IP4856CX25
- added U?: USB3320, symbol Zynq_UltraScale:USB3320
- added Y?: 24MHz, symbol Device:Crystal
Connections:
- net +1V0: now also R132.2; no longer R132.1
- net +1V8: now also C61.1, R118.1, U?.11 (REFSEL1), U?.14 (REFSEL2), U?.28 (VDD18), U?.30 (VDD18), U?.32 (VDDIO), U?.8 (REFSEL0), U?.B3 (VCCA), U?.B4 (VCC), U?.C2 (ENABLE)
- net +3V3: now also U?.21 (VBAT), U?.27 (RESETB), U?.A4 (VSUPPLY), U?.C4 (V_SD_REF); no longer C61.1, R118.1
- net CS: now also U?.C2 (S#)
- net D+: now also U?.18 (DP)
- net D-: now also U?.19 (DM)
- net GND: now also R132.1, C?.1, C?.2, C?.2, R?.1, U?.33 (CTR_GND), U?.B3 (VSS), U?.B4 (VLDO), U?.C3 (GND); no longer C53.1, R132.2
- net IO0: now also U?.D3 (DQ0)
- net IO1: now also U?.D2 (DQ1)
- net IO2: now also U?.C4 (W#/DQ2)
- net IO3: now also U?.D4 (DQ3)
- net SCK: now also U?.B2 (C)
- net SD_CLK: now also U?.C5 (CLK_SD)
- net SD_CMD: now also U?.C4 (V_SD_REF)
- net SD_D0: now also U?.D5 (DATA0_SD)
- net SD_D1: now also U?.E5 (DATA1_SD)
- net SD_D2: now also U?.A5 (DATA2_SD)
- net SD_D3: now also U?.B5 (DATA3_SD)
- net MIO_CD: now reaches U5.A11 (PS_MIO45)
- net MIO_CD: now also U?.D3 (CD)
- net MIO_DAT2: now reaches U5.A12 (PS_MIO48)
- net MIO_DAT2: now also U?.A1 (DATA2_H)
- net MIO_CMD: now reaches U5.A13 (PS_MIO50)
- net MIO_CMD: now also U?.D2 (CMD_H)
- net MIO_DIR0: now reaches U5.B10 (PS_MIO41)
- net MIO_DIR0: now also U?.A3 (DIR_0)
- net MIO_WP: now reaches U5.B11 (PS_MIO44)
- net MIO_WP: now also U?.E4 (WP)
- net MIO_DAT1: now reaches U5.B12 (PS_MIO47)
- net MIO_DAT1: now also U?.E1 (DATA1_H)
- net MIO_SEL: now reaches U5.C10 (PS_MIO39)
- net MIO_SEL: now also U?.B2 (SEL)
- net MIO_DAT0: now reaches U5.C12 (PS_MIO46)
- net MIO_DAT0: now also U?.D1 (DATA0_H)
- net MIO_CLK_IN: now reaches U5.C13 (PS_MIO51)
- net MIO_CLK_IN: now also U?.C1 (CLK_IN)
- net MIO_DIR_CMD: now reaches U5.D11 (PS_MIO40)
- net MIO_DIR_CMD: now also U?.A2 (DIR_CMD)
- net MIO_DIR1_3: now reaches U5.D12 (PS_MIO42)
- net MIO_DIR1_3: now also U?.E3 (DIR_1_3)
- net MIO_DAT3: now reaches U5.D13 (PS_MIO49)
- net MIO_DAT3: now also U?.B1 (DATA3_H)
- net MIO_USB_STP: now reaches U5.A14 (PS_MIO58)
- net MIO_USB_STP: now also U?.29 (STP)
- net MIO_USB_DATA1: now reaches U5.B14 (PS_MIO57)
- net MIO_USB_DATA1: now also U?.4 (DATA1)
- net MIO_USB_NXT: now reaches U5.C14 (PS_MIO55)
- net MIO_USB_NXT: now also U?.2 (NXT)
- net MIO_USB_DATA6: now reaches U5.C15 (PS_MIO62)
- net MIO_USB_DATA6: now also U?.10 (DATA6)
- net MIO_USB_DATA4: now reaches U5.D15 (PS_MIO60)
- net MIO_USB_DATA4: now also U?.7 (DATA4)
- net MIO_USB_DATA0: now reaches U5.E14 (PS_MIO56)
- net MIO_USB_DATA0: now also U?.3 (DATA0)
- net MIO_USB_DATA3: now reaches U5.E15 (PS_MIO59)
- net MIO_USB_DATA3: now also U?.6 (DATA3)
- net MIO_USB_DIR: now reaches U5.F14 (PS_MIO53)
- net MIO_USB_DIR: now also U?.31 (DIR)
- net MIO_USB_DATA7: now reaches U5.F16 (PS_MIO63)
- net MIO_USB_DATA7: now also U?.13 (DATA7)
- net MIO_USB_CLK: now reaches U5.G14 (PS_MIO52)
- net MIO_USB_CLK: now also U?.1 (CLKOUT)
- net MIO_USB_DATA2: now reaches U5.G15 (PS_MIO54)
- net MIO_USB_DATA2: now also U?.5 (DATA2)
- net MIO_USB_DATA5: now reaches U5.G16 (PS_MIO61)
- net MIO_USB_DATA5: now also U?.9 (DATA5)
- net RX: no longer names the net of U5.V5 (PS_MIO9)
- net TX: no longer names the net of U5.V3 (PS_MIO8)
- new net: U?.A2 (NC), U?.A3 (RFU), U?.A4 (RESET#), U?.A4Ç (RFU), U?.A5 (RFU), U?.B1 (RFU), U?.B5 (RFU), U?.C1 (RFU), U?.C3 (RFU), U?.C5 (RFU), U?.D1 (RFU), U?.D5 (RFU), U?.E1 (RFU), U?.E2 (RFU), U?.E3 (RFU), U?.E5 (RFU)
- new net: C?.2, U?.20 (VDD33), U?.23 (ID)
- new net: R?.2, U?.22 (VBUS)
- new net: R?.2, U?.24 (RBIAS)
- new net: C?.1, U?.25 (XO), Y?.2
- new net: C?.1, U?.26 (REFCLK), Y?.1
- new net +5C: U?.17 (CPEN)
- new net VBUS: C53.1, R?.1
- no-connect marks 134 -> 80
Other:
- moved on the sheet: C53, C61, D10, D11, J2, R110, R112, R115, R116, R117, R118, R120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

Commit message: update
Parts:
- removed R132: 200, symbol Device:R_US
- removed U10: TPS3106K33DBV, symbol Zynq_7000:TPS3106K33DBV
- added C51, C52, C54, C55: 0.1uF, symbol Device:C
- added D12, D13: DIODE, symbol Simulation_SPICE:DIODE
- added D14: f, symbol Device:LED_ALT
- added R128: 8k, symbol Device:R_US
- added R129, R130: 4.7k, symbol Device:R_US
- added SW11: SW_Push, symbol Switch:SW_Push
- added U11: MAX16025, symbol Zynq_UltraScale:MAX16025
- R115: value 820 -> 10k
- R116: value 1300 -> 10k
- R117: value 100K -> 8k
- R122: value 1k -> 10k
- R131: value 1k -> 261
- gave numbers to parts that had none: 9
Connections:
- net +1V2 is gone; now on net +3V3: R131.1
- net +1V8: now also R117.1, R129.2, R130.2
- net +3V3: now also R115.1, R116.1, C51.1, U11.1 (VCC); no longer R117.1
- net GND: now also C51.2, C52.2, C54.2, C55.2, D12.2 (K), D13.2 (K), R128.2, SW11.2, U11.13 (MR_B), U11.17 (EPAD), U11.4 (TOL), U11.5 (GND)
- net PS_POR_B: now also R129.1, U11.11 (OUT1); no longer R117.2
- net SRST_B: now also R130.1, U11.10 (OUT2); no longer R122.2, SW10.1
- net at R115.2: now also SW10.1, D12.1 (A), U11.6 (EN1); no longer R116.1
- net +1V0: no longer names the net of R131.2
- net +1V0: now also D14.2 (A); no longer R115.1
- net +5C renamed +5V
- new net: D14.1 (K), U11.12 (RESET_B)
- new net: C52.1, U11.14 (CRESET)
- new net: C54.1, U11.15 (CDLY2)
- new net: C55.1, U11.16 (CDLY1)
- new net: R117.2, R128.1, U11.2 (IN1), U11.3 (IN2)
- new net: D13.1 (A), R122.2, SW11.1, U11.7 (EN2)
- no-connect marks 80 -> 81
Other:
- moved on the sheet: D11, R122, R123, R124, R125, R126, SW10, U9

Commit message: upd
Parts:
- removed C62: 100nF, symbol Device:C
- removed R119: 4.7k, symbol Device:R_US
- removed X1: ASE-xxxMHz, Oscillator:Oscillator_SMD_Abracon_ASE-4Pin_3.2x2.5mm, symbol Oscillator:ASE-xxxMHz
- added C?: 0.01uF, symbol Device:C
- added R?: 4.7k, symbol Device:R_US
- added R?: 24.9k, symbol Device:R_US
- added U?: SiT8103AC-23-18E-33.33333, symbol Zynq_UltraScale:SiT8103AC-23-18E-33.33333
Connections:
- net +1V8: now also R120.1, R123.1, R125.1, R126.1, C?.2, R?.2, U?.~ (VCC)
- net +3V3: no longer R120.1, R123.1, R125.1, R126.1
- net GND: now also C?.1, U?.~ (VCC)
- net PS_CLK: now also R?.1
- new net: R?.1, U?.~ (VCC)
- new net: R?.2, U?.~ (VCC)
Other:
- note added: "SPI FLASH\n"
- note removed: "QUAD SPI FLASH\n"
Changed lines of the file:
@@
-$EndComp
-$Comp
-L Oscillator:ASE-xxxMHz X1
-U 1 1 616D82E4
-P 10500 10200
-F 0 "X1" H 10600 10450 50  0000 L CNN
-F 1 "ASE-xxxMHz" H 10600 9950 50  0000 L CNN
-F 2 "Oscillator:Oscillator_SMD_Abracon_ASE-4Pin_3.2x2.5mm" H 11200 9850 50  0001 C CNN
-F 3 "http://www.abracon.com/Oscillators/ASV.pdf" H 10400 10200 50  0001 C CNN
-	1    10500 10200
-	1    0    0    -1
 $EndComp
 $Comp
@@
 Wire Wire Line
 	3750 8200 3750 7800
-$Comp
-L Device:R_US R119
-U 1 1 6176CF65
-P 9950 9950
-F 0 "R119" H 10018 9996 50  0000 L CNN
-F 1 "4.7k" H 10018 9905 50  0000 L CNN
-F 2 "" V 9990 9940 50  0001 C CNN
-F 3 "~" H 9950 9950 50  0001 C CNN
-	1    9950 9950
-	1    0    0    -1
-$EndComp
-$Comp
-L Device:C C62
-U 1 1 6176D7DD
-P 10800 9750
-F 0 "C62" V 10548 9750 50  0000 C CNN
-F 1 "100nF" V 10639 9750 50  0000 C CNN
-F 2 "" H 10838 9600 50  0001 C CNN
-F 3 "~" H 10800 9750 50  0001 C CNN
-	1    10800 9750
-	0    1    1    0
-$EndComp
-Wire Wire Line
-	10200 10200 9950 10200
-Wire Wire Line
-	9950 10200 9950 10100
-Wire Wire Line
-	9950 9800 9950 9750
-Wire Wire Line
-	9950 9750 10500 9750
-Wire Wire Line
-	10500 9900 10500 9750
-Connection ~ 10500 9750
-Wire Wire Line
-	10500 9750 10650 9750
 NoConn ~ 13500 8350
 $Comp
@@
 Wire Wire Line
 	7600 6400 7600 6350
-$Comp
-L power:+3V3 #PWR0223
-U 1 1 6185F306
-P 11800 4450
-F 0 "#PWR0223" H 11800 4300 50  0001 C CNN
-F 1 "+3V3" H 11800 4623 50  0000 C CNN
-F 2 "" H 11800 4450 50  0001 C CNN
-F 3 "" H 11800 4450 50  0001 C CNN
-	1    11800 4450
-	1    0    0    -1
-$EndComp
 Wire Wire Line
 	11800 4450 11800 4750
@@
 Wire Wire Line
 	9250 10950 9100 10950
-$Comp
-L power:GND #PWR0225
-U 1 1 61882F33
-P 10500 10650
-F 0 "#PWR0225" H 10500 10400 50  0001 C CNN
-F 1 "GND" H 10500 10477 50  0000 C CNN
-F 2 "" H 10500 10650 50  0001 C CNN
-F 3 "" H 10500 10650 50  0001 C CNN
-	1    10500 10650
-	1    0    0    -1
-$EndComp
-Wire Wire Line
-	10500 10650 10500 10500
-$Comp
-L power:GND #PWR0226
-U 1 1 618883A0
-P 11100 9800
-F 0 "#PWR0226" H 11100 9550 50  0001 C CNN
-F 1 "GND" H 11100 9627 50  0000 C CNN
-F 2 "" H 11100 9800 50  0001 C CNN
-F 3 "" H 11100 9800 50  0001 C CNN
-	1    11100 9800
-	1    0    0    -1
-$EndComp
-Wire Wire Line
-	11100 9800 11100 9750
-Wire Wire Line
-	11100 9750 10950 9750
-$Comp
-L power:+3V3 #PWR0229
-U 1 1 61899B93
-P 10500 9550
-F 0 "#PWR0229" H 10500 9400 50  0001 C CNN
-F 1 "+3V3" H 10500 9723 50  0000 C CNN
-F 2 "" H 10500 9550 50  0001 C CNN
-F 3 "" H 10500 9550 50  0001 C CNN
-	1    10500 9550
-	1    0    0    -1
-$EndComp
-Wire Wire Line
-	10500 9550 10500 9750
 Wire Wire Line
 	8950 1750 9150 1750
@@
 Text Label 14000 7750 2    50   ~ 0
 PS_TMS
-Text Label 11200 10200 2    50   ~ 0
+Text Label 11700 10300 2    50   ~ 0
 PS_CLK
 Wire Wire Line
-	10800 10200 11200 10200
+	11400 10300 11700 10300
 Text Label 14000 8650 2    50   ~ 0
 PS_CLK
@@
 XCZU2CG\n\n
 Text Notes 6900 950  0    118  ~ 24
-QUAD SPI FLASH\n
+SPI FLASH\n
 Text Notes 6450 9400 0    118  ~ 24
 SD\n
@@
 Wire Wire Line
 	8300 6900 8300 6250
+$Comp
+L power:+1V8 #PWR?
+U 1 1 613B492B
+P 11800 4450
+F 0 "#PWR?" H 11800 4300 50  0001 C CNN
+F 1 "+1V8" H 11815 4623 50  0000 C CNN
+F 2 "" H 11800 4450 50  0001 C CNN
+F 3 "" H 11800 4450 50  0001 C CNN
+	1    11800 4450
+	1    0    0    -1
+$EndComp
+$Comp
+L Zynq_UltraScale:SiT8103AC-23-18E-33.33333 U?
+U 1 1 613F8AF9
+P 10650 10150
+F 0 "U?" H 10650 10515 50  0000 C CNN
+F 1 "SiT8103AC-23-18E-33.33333" H 11000 9750 50  0000 C CNN
+F 2 "" H 10650 10650 50  0001 C CNN
+F 3 "" H 10650 10650 50  0001 C CNN
+	1    10650 10150
+	1    0    0    -1
+$EndComp
+$Comp
+L Device:R_US R?
+U 1 1 613F8B84
+P 10200 10050
+F 0 "R?" V 10100 10000 50  0000 L CNN
+F 1 "4.7k" V 10268 10005 50  0000 L CNN
+F 2 "" V 10240 10040 50  0001 C CNN
+F 3 "~" H 10200 10050 50  0001 C CNN
+	1    10200 10050
+	0    1    1    0
+$EndComp
+$Comp
+L power:GND #PWR?
+U 1 1 613F93C0
+P 10200 10400
+F 0 "#PWR?" H 10200 10150 50  0001 C CNN
+F 1 "GND" H 10200 10227 50  0000 C CNN
+F 2 "" H 10200 10400 50  0001 C CNN
+F 3 "" H 10200 10400 50  0001 C CNN
+	1    10200 10400
+	1    0    0    -1
+$EndComp
+$Comp
+L power:+1V8 #PWR?
+U 1 1 61414997
+P 11300 10050
+F 0 "#PWR?" H 11300 9900 50  0001 C CNN
+F 1 "+1V8" V 11315 10178 50  0000 L CNN
+F 2 "" H 11300 10050 50  0001 C CNN
+F 3 "" H 11300 10050 50  0001 C CNN
+	1    11300 10050
+	0    1    -1   0
+$EndComp
+Wire Wire Line
+	11300 10050 11000 10050
+Wire Wire Line
+	10350 10300 10200 10300
+Wire Wire Line
+	10200 10300 10200 10400
+$Comp
+L power:+1V8 #PWR?
+U 1 1 6148BC24
+P 10000 10050
+F 0 "#PWR?" H 10000 9900 50  0001 C CNN
+F 1 "+1V8" V 10015 10178 50  0000 L CNN
+F 2 "" H 10000 10050 50  0001 C CNN
+F 3 "" H 10000 10050 50  0001 C CNN
+	1    10000 10050
+	0    -1   1    0
+$EndComp
+Wire Wire Line
+	10050 10050 10000 10050
+$Comp
+L Device:C C?
+U 1 1 614E2091
+P 11250 9750
+F 0 "C?" V 10998 9750 50  0000 C CNN
+F 1 "0.01uF" V 11089 9750 50  0000 C CNN
+F 2 "" H 11288 9600 50  0001 C CNN
+F 3 "~" H 11250 9750 50  0001 C CNN
+	1    11250 9750
+	0    1    1    0
+$EndComp
+Wire Wire Line
+	11100 9750 11000 9750
+Wire Wire Line
+	11000 9750 11000 10050
+Connection ~ 11000 10050
+Wire Wire Line
+	11000 10050 10950 10050
+$Comp
+L power:GND #PWR?
+U 1 1 61500952
+P 11500 9750
+F 0 "#PWR?" H 11500 9500 50  0001 C CNN
+F 1 "GND" H 11500 9577 50  0000 C CNN
+F 2 "" H 11500 9750 50  0001 C CNN
+F 3 "" H 11500 9750 50  0001 C CNN
+	1    11500 9750
+	0    -1   -1   0
+$EndComp
+Wire Wire Line
+	11500 9750 11400 9750
+$Comp
+L Device:R_US R?
+U 1 1 6151F3DC
+P 11250 10300
+F 0 "R?" V 11150 10250 50  0000 L CNN
+F 1 "24.9k" V 11318 10255 50  0000 L CNN
+F 2 "" V 11290 10290 50  0001 C CNN
+F 3 "~" H 11250 10300 50  0001 C CNN
+	1    11250 10300
+	0    1    1    0
+$EndComp
+Wire Wire Line
+	11100 10300 10950 10300
 $EndSCHEMATC
